Commit message: Update marsyard2021.world.xacro

File: blender_gazebo/worlds/marsyard2021.world.xacro (robot description, xacro)
@@ -34,32 +34,4 @@
       <uri>model://ground_plane</uri>
     </include>
-    <!-- Actors is model with automated moving models in gazebo in this cas our actor is cosmonaut named Lagari Hasan Çelebi.-->
-    <actor name="Lâgari Hasan Çelebi">
-      <link name="cosmonaut">
-        <visual name="visual">
-          <pose>0 25 0.9 0 0 1.57</pose>
-          <geometry>
-            <mesh>
-              <scale>1 1 1</scale>
-              <uri>/home/baran/rover_simulation_ws/src/Simulations/blender_gazebo/worlds/cosmonaut-dae/cosmonaut.dae</uri> <!-- Change this path if you want cosmounaut you can use pwd command on terminal.-->
-            </mesh>
-          </geometry>
-        </visual>
-      </link>
-      <script>
-        <loop>true</loop>
-        <auto_start>true</auto_start>
-        <trajectory id="0" type="square">
-          <waypoint>
-            <time>0.0</time>
-            <pose>-1 -1 0 0 0 0</pose>
-          </waypoint>
-          <waypoint>
-            <time>30.0</time>
-            <pose>20 -1 0 0 0 0</pose>
-          </waypoint>
-        </trajectory>
-      </script>
-    </actor>
     <xacro:include filename="$(find blender_gazebo)/sdf/landmark.sdf.xacro"/>
     <!-- Artag ids from 1 to 15-->
